File: hardware/lan64usb.sch (KiCad schematic (older format))
At the start: 18 parts, among them J1 USB_B, J2 ISP, J3 C64_Userport, U1 ATMEGA8-16PU, Y1 Crystal 12MHz

Commit message: Alle Footprints zugeordnet und Net Liste erstellt.
Parts:
- C1: footprint (none) -> w_capacitors:CP_5x11mm
- C2, C3: footprint (none) -> Capacitors_THT:C_Disc_D4.7mm_W2.5mm_P5.00mm
- C4, C5: footprint (none) -> Capacitors_THT:C_Disc_D3.8mm_W2.6mm_P2.50mm
- D1: footprint (none) -> w_indicators:led_3mm_green
- D2, D3: footprint (none) -> Diodes_THT:D_DO-35_SOD27_P7.62mm_Horizontal
- J1: footprint (none) -> Connectors:USB_B
- J2: footprint (none) -> w_conn_strip:vasch_strip_3x2
- J3: footprint (none) -> ka_c64:c64_userport
- R1, R2, R3, R4, R5: footprint (none) -> Resistors_THT:R_Axial_DIN0207_L6.3mm_D2.5mm_P10.16mm_Horizontal
- U1: footprint DIL28 -> w_pth_circuits:dil_28-300_socket
- Y1: footprint (none) -> Crystals:Crystal_HC49-4H_Vertical
Changed lines of the file:
@@
 F 0 "R4" V 1980 2550 50  0000 C CNN
 F 1 "10k" V 1900 2550 50  0000 C CNN
-F 2 "" V 1830 2550 50  0001 C CNN
+F 2 "Resistors_THT:R_Axial_DIN0207_L6.3mm_D2.5mm_P10.16mm_Horizontal" V 1830 2550 50  0001 C CNN
 F 3 "" H 1900 2550 50  0001 C CNN
 	1    1900 2550
@@
 F 0 "Y1" H 2100 3500 50  0000 C CNN
 F 1 "Crystal 12MHz" V 1850 3450 50  0000 C CNN
-F 2 "" H 2100 3350 50  0001 C CNN
+F 2 "Crystals:Crystal_HC49-4H_Vertical" H 2100 3350 50  0001 C CNN
 F 3 "" H 2100 3350 50  0001 C CNN
 	1    2100 3350
@@
 F 0 "C2" H 1725 3250 50  0000 L CNN
 F 1 "22p" H 1725 3050 50  0000 L CNN
-F 2 "" H 1738 3000 50  0001 C CNN
+F 2 "Capacitors_THT:C_Disc_D4.7mm_W2.5mm_P5.00mm" H 1738 3000 50  0001 C CNN
 F 3 "" H 1700 3150 50  0001 C CNN
 	1    1700 3150
@@
 F 0 "C3" H 1725 3650 50  0000 L CNN
 F 1 "22p" H 1725 3450 50  0000 L CNN
-F 2 "" H 1738 3400 50  0001 C CNN
+F 2 "Capacitors_THT:C_Disc_D4.7mm_W2.5mm_P5.00mm" H 1738 3400 50  0001 C CNN
 F 3 "" H 1700 3550 50  0001 C CNN
 	1    1700 3550
@@
 F 0 "D1" H 9400 1200 50  0000 C CNN
 F 1 "LED" H 9400 1000 50  0000 C CNN
-F 2 "" H 9400 1100 50  0001 C CNN
+F 2 "w_indicators:led_3mm_green" H 9400 1100 50  0001 C CNN
 F 3 "" H 9400 1100 50  0001 C CNN
 	1    9400 1100
@@
 F 0 "R1" V 8830 1100 50  0000 C CNN
 F 1 "100" V 8750 1100 50  0000 C CNN
-F 2 "" V 8680 1100 50  0001 C CNN
+F 2 "Resistors_THT:R_Axial_DIN0207_L6.3mm_D2.5mm_P10.16mm_Horizontal" V 8680 1100 50  0001 C CNN
 F 3 "" H 8750 1100 50  0001 C CNN
 	1    8750 1100
@@
 F 0 "C4" H 1475 7350 50  0000 L CNN
 F 1 "100n" H 1475 7150 50  0000 L CNN
-F 2 "" H 1488 7100 50  0001 C CNN
+F 2 "Capacitors_THT:C_Disc_D3.8mm_W2.6mm_P2.50mm" H 1488 7100 50  0001 C CNN
 F 3 "" H 1450 7250 50  0001 C CNN
 	1    1450 7250
@@
 F 0 "C5" H 1775 7350 50  0000 L CNN
 F 1 "100n" H 1775 7150 50  0000 L CNN
-F 2 "" H 1788 7100 50  0001 C CNN
+F 2 "Capacitors_THT:C_Disc_D3.8mm_W2.6mm_P2.50mm" H 1788 7100 50  0001 C CNN
 F 3 "" H 1750 7250 50  0001 C CNN
 	1    1750 7250
@@
 F 0 "J1" H 7950 2700 50  0000 L CNN
 F 1 "USB_B" H 7950 2600 50  0000 L CNN
-F 2 "" H 8300 2200 50  0001 C CNN
+F 2 "Connectors:USB_B" H 8300 2200 50  0001 C CNN
 F 3 "" H 8300 2200 50  0001 C CNN
 	1    8150 2250
@@
 F 0 "R2" V 9630 2250 50  0000 C CNN
 F 1 "68" V 9550 2250 50  0000 C CNN
-F 2 "" V 9480 2250 50  0001 C CNN
+F 2 "Resistors_THT:R_Axial_DIN0207_L6.3mm_D2.5mm_P10.16mm_Horizontal" V 9480 2250 50  0001 C CNN
 F 3 "" H 9550 2250 50  0001 C CNN
 	1    9550 2250
@@
 F 0 "R3" V 9630 2450 50  0000 C CNN
 F 1 "68" V 9550 2450 50  0000 C CNN
-F 2 "" V 9480 2450 50  0001 C CNN
+F 2 "Resistors_THT:R_Axial_DIN0207_L6.3mm_D2.5mm_P10.16mm_Horizontal" V 9480 2450 50  0001 C CNN
 F 3 "" H 9550 2450 50  0001 C CNN
 	1    9550 2450
@@
 F 0 "D2" H 8700 2850 50  0000 C CNN
 F 1 "ZD 3,6" H 8700 2650 50  0000 C CNN
-F 2 "" H 8700 2750 50  0001 C CNN
+F 2 "Diodes_THT:D_DO-35_SOD27_P7.62mm_Horizontal" H 8700 2750 50  0001 C CNN
 F 3 "" H 8700 2750 50  0001 C CNN
 	1    8700 2750
@@
 F 0 "D3" H 9000 2850 50  0000 C CNN
 F 1 "ZD 3,6" H 9000 2650 50  0000 C CNN
-F 2 "" H 9000 2750 50  0001 C CNN
+F 2 "Diodes_THT:D_DO-35_SOD27_P7.62mm_Horizontal" H 9000 2750 50  0001 C CNN
 F 3 "" H 9000 2750 50  0001 C CNN
 	1    9000 2750
@@
 F 0 "R5" V 9330 2750 50  0000 C CNN
 F 1 "2,2k" V 9250 2750 50  0000 C CNN
-F 2 "" V 9180 2750 50  0001 C CNN
+F 2 "Resistors_THT:R_Axial_DIN0207_L6.3mm_D2.5mm_P10.16mm_Horizontal" V 9180 2750 50  0001 C CNN
 F 3 "" H 9250 2750 50  0001 C CNN
 	1    9250 2750
@@
 F 0 "C1" H 9075 3200 50  0000 L CNN
 F 1 "10µ" H 9075 3000 50  0000 L CNN
-F 2 "" H 9088 2950 50  0001 C CNN
+F 2 "w_capacitors:CP_5x11mm" H 9088 2950 50  0001 C CNN
 F 3 "" H 9050 3100 50  0001 C CNN
 	1    9050 3100
@@
 F 0 "J2" H 8850 4450 50  0000 C CNN
 F 1 "ISP" H 8850 4050 50  0000 C CNN
-F 2 "" H 8800 4250 50  0001 C CNN
+F 2 "w_conn_strip:vasch_strip_3x2" H 8800 4250 50  0001 C CNN
 F 3 "" H 8800 4250 50  0001 C CNN
 	1    8800 4250
@@
 F 0 "J3" H 9050 6400 60  0000 C CNN
 F 1 "C64_Userport" H 9050 5000 60  0000 C CNN
-F 2 "" V 9000 6050 60  0001 C CNN
+F 2 "ka_c64:c64_userport" V 9000 6050 60  0001 C CNN
 F 3 "" V 9000 6050 60  0001 C CNN
 	1    9050 5700
@@
 F 0 "U1" H 2750 4950 50  0000 L BNN
 F 1 "ATMEGA8-16PU" H 4000 2200 50  0000 L BNN
-F 2 "DIL28" H 3500 3650 50  0001 C CIN
+F 2 "w_pth_circuits:dil_28-300_socket" H 3500 3650 50  0001 C CIN
 F 3 "" H 3500 3650 50  0001 C CNN
 	1    3500 3650
