File: hardware/lan64usb.kicad_pcb (KiCad board)
At the start: 2 copper layers, 77.5 x 34.3 mm, 19 parts, among them J1 USB_B, J2 ISP, J3 C64_Userport, U1 ATMEGA8-16PU, Y1 Crystal 12MHz

Commit message: 3D Ansicht hinzugefügt. Stecker fehlt noch!
Other:
- board text added: "lan64usb Rev.: 1.2.0"
- board text removed: "Lan64USB Rev: 1.2.0"
Changed lines of the file:
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@@
     (links 51)
     (no_connects 0)
-    (area 110.414999 75.489999 188.035001 109.930001)
+    (area 109.619999 75.489999 189.0466 110.305)
     (thickness 1.6)
     (drawings 6)
@@
     (effects (font (size 1.5 1.5) (thickness 0.3)))
   )
-  (gr_text "Lan64USB\nRev: 1.2.0" (at 179.705 79.375) (layer F.SilkS)
+  (gr_text "lan64usb\nRev.: 1.2.0" (at 179.705 79.375) (layer F.SilkS)
     (effects (font (size 1.5 1.5) (thickness 0.3)))
   )
